Commit message: 🚗 Update README and URDF to make a for wheel robot

File: description/gazebo_control.xacro (robot description, xacro)
@@ -4,12 +4,18 @@
         <plugin name="diff_drive" filename="libgazebo_ros_diff_drive.so">
             <!-- WHEEL INFORMATION -->
+            <!-- Two wheel pairs: front + rear -->
+            <num_wheel_pairs>2</num_wheel_pairs>
             <left_joint>left_wheel_joint</left_joint>
+            <left_joint>left_front_wheel_joint</left_joint>
             <right_joint>right_wheel_joint</right_joint>
+            <right_joint>right_front_wheel_joint</right_joint>
             <wheel_separation>0.35</wheel_separation>
+            <wheel_separation>0.35</wheel_separation>
+            <wheel_diameter>0.1</wheel_diameter>
             <wheel_diameter>0.1</wheel_diameter>
             <!-- LIMITS -->
             <max_wheel_torque>200</max_wheel_torque>
             <max_wheel_acceleration>10.0</max_wheel_acceleration>
-            <!-- OUTPUTS-->
+            <!-- OUTPUTS -->
             <odometry_frame>odom</odometry_frame>
             <robot_base_frame>base_link</robot_base_frame>

File: description/robot_core.xacro (robot description, xacro)
@@ -101,6 +101,62 @@
         <material>Gazebo/Black</material>
     </gazebo>
+    <!-- ==================== ADDITIONAL LEFT WHEEL LINK ====================  -->
+    <link name="left_front_wheel">
+        <visual>
+            <origin xyz="0 0 0" rpy="0 0 0"/>
+            <geometry>
+                <cylinder radius="0.05" length="0.04"/>
+            </geometry>
+            <material name="black"/>
+        </visual>
+        <collision>
+            <origin xyz="0 0 0" rpy="0 0 0"/>
+            <geometry>
+                <cylinder radius="0.05" length="0.04"/>
+            </geometry>
+        </collision>
+        <xacro:inertial_cylinder mass="0.1" radius="0.05" length="0.04">
+            <origin xyz="0 0 0" rpy="0 0 0"/>
+        </xacro:inertial_cylinder>
+    </link>
+    <joint name="left_front_wheel_joint" type="continuous">
+        <parent link="base_link"/>
+        <child link="left_front_wheel"/>
+        <origin xyz="0.2 0.175 0" rpy="-${pi/2} 0 0"/>
+        <axis xyz="0 0 1"/>
+    </joint>
+    <gazebo reference="left_front_wheel">
+        <material>Gazebo/Black</material>
+    </gazebo>
+    <!-- ==================== ADDITIONAL RIGHT WHEEL LINK ====================  -->
+    <link name="right_front_wheel">
+        <visual>
+            <origin xyz="0 0 0" rpy="0 0 0"/>
+            <geometry>
+                <cylinder radius="0.05" length="0.04"/>
+            </geometry>
+            <material name="black"/>
+        </visual>
+        <collision>
+            <origin xyz="0 0 0" rpy="0 0 0"/>
+            <geometry>
+                <cylinder radius="0.05" length="0.04"/>
+            </geometry>
+        </collision>
+        <xacro:inertial_cylinder mass="0.1" radius="0.05" length="0.04">
+            <origin xyz="0 0 0" rpy="0 0 0"/>
+        </xacro:inertial_cylinder>
+    </link>
+    <joint name="right_front_wheel_joint" type="continuous">
+        <parent link="base_link"/>
+        <child link="right_front_wheel"/>
+        <origin xyz="0.2 -0.175 0" rpy="${pi/2} 0 0"/>
+        <axis xyz="0 0 -1"/>
+    </joint>
+    <gazebo reference="right_front_wheel">
+        <material>Gazebo/Black</material>
+    </gazebo>
     <!-- ==================== CASTER WHEEL LINK ====================  -->
-    <joint name="caster_wheel_joint" type="fixed">
+    <!-- <joint name="caster_wheel_joint" type="fixed">
         <parent link="chassis"/>
         <child link="caster_wheel"/>
@@ -129,4 +185,4 @@
         <mu2 value="0.001"/>
         <material>Gazebo/Black</material>
-    </gazebo>
+    </gazebo> -->
 </robot>
