Commit message: ✨ Add Gazebo control and launch files for robot simulation

File: description/robot_core.xacro (robot description, xacro)
@@ -42,4 +42,7 @@
         </xacro:inertial_box>
     </link>
+    <gazebo reference="chassis">
+        <material>Gazebo/White</material>
+    </gazebo>
     <!-- ==================== LEFT WHEEL LINK ====================  -->
     <link name="left_wheel">
@@ -67,4 +70,7 @@
         <axis xyz="0 0 1"/>
     </joint>
+    <gazebo reference="left_wheel">
+        <material>Gazebo/Black</material>
+    </gazebo>
     <!-- ==================== RIGHT WHEEL LINK ====================  -->
     <link name="right_wheel">
@@ -92,4 +98,7 @@
         <axis xyz="0 0 -1"/>
     </joint>
+    <gazebo reference="right_wheel">
+        <material>Gazebo/Black</material>
+    </gazebo>
     <!-- ==================== CASTER WHEEL LINK ====================  -->
     <joint name="caster_wheel_joint" type="fixed">
@@ -116,3 +125,8 @@
         </xacro:inertial_sphere>
     </link>
+    <gazebo reference="caster_wheel">
+        <mu1 value="0.001"/>
+        <mu2 value="0.001"/>
+        <material>Gazebo/Black</material>
+    </gazebo>
 </robot>

Commit message: 🚨 Add lidar.xacro file and include in robot.urdf.xacro; define laser joint and frame

File: description/robot_core.xacro (robot description, xacro)
@@ -14,4 +14,7 @@
     <material name="black">
         <color rgba="0 0 0 1"/>
+    </material>
+    <material name="red">
+        <color rgba="1 0 0 1"/>
     </material>
     <!-- ==================== BASE LINK ====================  -->
